File: bms-breakout/battery-balance-connector/battery-balance-connector.kicad_sch (KiCad schematic)
At the start: 10 parts, among them J1 Conn_01x04, J10 Conn_01x01, J2 Conn_01x04, J3 Conn_01x01, J4 Conn_01x01, J5 Conn_01x01, J6 Conn_01x01, J7 Conn_01x01, J8 Conn_01x01, J9 Conn_01x01

Commit message: made some more progress on the battery balance connector
Parts:
- J10, J3, J4, J5, J6, J7, J8, J9: footprint (none) -> Connector_Wire:SolderWire-1sqmm_1x01_D1.4mm_OD2.7mm_Relief
Connections:
- net CELL1: now also J2.3 (Pin_3); no longer J2.2 (Pin_2)
- net CELL2: now also J2.2 (Pin_2); no longer J2.3 (Pin_3)
- net CELL3: now also J2.1 (Pin_1); no longer J2.4 (Pin_4)
- net GND: now also J2.4 (Pin_4); no longer J2.1 (Pin_1)
Changed lines of the file:
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@@
-    (stroke (width 0) (type default))
-  )
-  (wire (pts (xy 19.05 40.64) (xy 19.05 44.45))
     (stroke (width 0) (type default))
   )
@@
     (stroke (width 0) (type default))
   )
-  (wire (pts (xy 19.05 40.64) (xy 30.48 40.64))
-    (stroke (width 0) (type default))
-  )
   (wire (pts (xy 73.66 33.02) (xy 81.28 33.02))
     (stroke (width 0) (type default))
@@
     (stroke (width 0) (type default))
   )
+  (wire (pts (xy 25.4 48.26) (xy 25.4 50.8))
+    (stroke (width 0) (type default))
+  )
+  (wire (pts (xy 25.4 40.64) (xy 30.48 40.64))
+    (stroke (width 0) (type default))
+  )
   (wire (pts (xy 73.66 43.18) (xy 81.28 43.18))
     (stroke (width 0) (type default))
@@
     (effects (font (size 1.27 1.27)) (justify left bottom))
   )
-  (label "CELL1" (at 25.4 43.18 0) (fields_autoplaced)
-    (effects (font (size 1.27 1.27)) (justify left bottom))
-  )
-  (label "CELL2" (at 25.4 45.72 0) (fields_autoplaced)
-    (effects (font (size 1.27 1.27)) (justify left bottom))
-  )
   (label "CELL2" (at 73.66 43.18 0) (fields_autoplaced)
     (effects (font (size 1.27 1.27)) (justify left bottom))
@@
     (effects (font (size 1.27 1.27)) (justify left bottom))
   )
+  (label "CELL1" (at 25.4 45.72 0) (fields_autoplaced)
+    (effects (font (size 1.27 1.27)) (justify left bottom))
+  )
+  (label "CELL3" (at 25.4 40.64 0) (fields_autoplaced)
+    (effects (font (size 1.27 1.27)) (justify left bottom))
+  )
   (label "CELL4" (at 73.66 33.02 0) (fields_autoplaced)
     (effects (font (size 1.27 1.27)) (justify left bottom))
@@
     (effects (font (size 1.27 1.27)) (justify left bottom))
   )
+  (label "CELL2" (at 25.4 43.18 0) (fields_autoplaced)
+    (effects (font (size 1.27 1.27)) (justify left bottom))
+  )
   (label "CELL6" (at 73.66 22.86 0) (fields_autoplaced)
     (effects (font (size 1.27 1.27)) (justify left bottom))
@@
     (effects (font (size 1.27 1.27)) (justify left bottom))
   )
-  (label "CELL3" (at 25.4 48.26 0) (fields_autoplaced)
-    (effects (font (size 1.27 1.27)) (justify left bottom))
-  )
   (label "CELL6" (at 25.4 26.67 0) (fields_autoplaced)
     (effects (font (size 1.27 1.27)) (justify left bottom))
@@
       (effects (font (size 1.27 1.27)) (justify left))
     )
-    (property "Footprint" "" (at 86.36 38.1 0)
+    (property "Footprint" "Connector_Wire:SolderWire-1sqmm_1x01_D1.4mm_OD2.7mm_Relief" (at 86.36 38.1 0)
       (effects (font (size 1.27 1.27)) hide)
     )
@@
       (effects (font (size 1.27 1.27)) (justify left))
     )
-    (property "Footprint" "" (at 86.36 48.26 0)
+    (property "Footprint" "Connector_Wire:SolderWire-1sqmm_1x01_D1.4mm_OD2.7mm_Relief" (at 86.36 48.26 0)
       (effects (font (size 1.27 1.27)) hide)
     )
@@
       (effects (font (size 1.27 1.27)) (justify left))
     )
-    (property "Footprint" "" (at 86.36 33.02 0)
+    (property "Footprint" "Connector_Wire:SolderWire-1sqmm_1x01_D1.4mm_OD2.7mm_Relief" (at 86.36 33.02 0)
       (effects (font (size 1.27 1.27)) hide)
     )
@@
       (effects (font (size 1.27 1.27)) (justify left))
     )
-    (property "Footprint" "" (at 86.36 22.86 0)
+    (property "Footprint" "Connector_Wire:SolderWire-1sqmm_1x01_D1.4mm_OD2.7mm_Relief" (at 86.36 22.86 0)
       (effects (font (size 1.27 1.27)) hide)
     )
@@
       (effects (font (size 1.27 1.27)) (justify left))
     )
-    (property "Footprint" "" (at 86.36 27.94 0)
+    (property "Footprint" "Connector_Wire:SolderWire-1sqmm_1x01_D1.4mm_OD2.7mm_Relief" (at 86.36 27.94 0)
       (effects (font (size 1.27 1.27)) hide)
     )
@@
       (effects (font (size 1.27 1.27)) (justify left))
     )
-    (property "Footprint" "" (at 86.36 17.78 0)
+    (property "Footprint" "Connector_Wire:SolderWire-1sqmm_1x01_D1.4mm_OD2.7mm_Relief" (at 86.36 17.78 0)
       (effects (font (size 1.27 1.27)) hide)
     )
@@
     )
   )
-  (symbol (lib_id "power:GND") (at 19.05 44.45 0) (unit 1)
-    (in_bom yes) (on_board yes) (dnp no) (fields_autoplaced)
-    (property "Reference" "#PWR01" (at 19.05 50.8 0)
-      (effects (font (size 1.27 1.27)) hide)
-    )
-    (property "Value" "GND" (at 19.05 49.53 0)
+  (symbol (lib_id "power:GND") (at 25.4 50.8 0) (unit 1)
+    (in_bom yes) (on_board yes) (dnp no) (fields_autoplaced)
+    (property "Reference" "#PWR01" (at 25.4 57.15 0)
+      (effects (font (size 1.27 1.27)) hide)
+    )
+    (property "Value" "GND" (at 25.4 55.88 0)
       (effects (font (size 1.27 1.27)))
     )
-    (property "Footprint" "" (at 19.05 44.45 0)
-      (effects (font (size 1.27 1.27)) hide)
-    )
-    (property "Datasheet" "" (at 19.05 44.45 0)
+    (property "Footprint" "" (at 25.4 50.8 0)
+      (effects (font (size 1.27 1.27)) hide)
+    )
+    (property "Datasheet" "" (at 25.4 50.8 0)
       (effects (font (size 1.27 1.27)) hide)
     )
@@
       (effects (font (size 1.27 1.27)) (justify left))
     )
-    (property "Footprint" "" (at 86.36 43.18 0)
+    (property "Footprint" "Connector_Wire:SolderWire-1sqmm_1x01_D1.4mm_OD2.7mm_Relief" (at 86.36 43.18 0)
       (effects (font (size 1.27 1.27)) hide)
     )
@@
       (effects (font (size 1.27 1.27)) (justify left))
     )
-    (property "Footprint" "" (at 86.36 53.34 0)
-      (effects (font (size 1.27 1.27)) hide)
-    )
+    (property "Footprint" "Connector_Wire:SolderWire-1sqmm_1x01_D1.4mm_OD2.7mm_Relief" (at 86.36 53.34 0)
+      (effects (font (size 1.27 1.27)) hide)
+    )

Commit message: V1.0.0 of battery balance connector
Parts:
- J10, J3, J4, J5, J6, J7, J8, J9: footprint Connector_Wire:SolderWire-1sqmm_1x01_D1.4mm_OD2.7mm_Relief -> Connector_Wire:SolderWirePad_1x01_SMD_2x4mm_2.7mmRelief
Changed lines of the file:
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@@
 (kicad_sch (version 20230121) (generator eeschema)
   (paper "A4")
+  (wire (pts (xy 25.4 45.72) (xy 30.48 45.72))
+    (stroke (width 0) (type default))
+  )
+  (wire (pts (xy 73.66 48.26) (xy 81.28 48.26))
+    (stroke (width 0) (type default))
+  )
+  (wire (pts (xy 25.4 29.21) (xy 30.48 29.21))
+    (stroke (width 0) (type default))
+  )
+  (polyline (pts (xy 12.7 60.96) (xy 52.07 60.96))
+    (stroke (width 0) (type default))
+  )
+  (polyline (pts (xy 104.14 12.7) (xy 104.14 60.96))
+    (stroke (width 0) (type default))
+  )
+  (wire (pts (xy 25.4 43.18) (xy 30.48 43.18))
+    (stroke (width 0) (type default))
+  )
+  (wire (pts (xy 73.66 33.02) (xy 81.28 33.02))
+    (stroke (width 0) (type default))
+  )
+  (polyline (pts (xy 52.07 12.7) (xy 52.07 60.96))
+    (stroke (width 0) (type default))
+  )
+  (wire (pts (xy 73.66 38.1) (xy 81.28 38.1))
+    (stroke (width 0) (type default))
+  )
   (wire (pts (xy 81.28 53.34) (xy 74.93 53.34))
     (stroke (width 0) (type default))
   )
-  (wire (pts (xy 25.4 45.72) (xy 30.48 45.72))
-    (stroke (width 0) (type default))
-  )
-  (wire (pts (xy 73.66 48.26) (xy 81.28 48.26))
+  (wire (pts (xy 25.4 26.67) (xy 30.48 26.67))
+    (stroke (width 0) (type default))
+  )
+  (wire (pts (xy 25.4 48.26) (xy 25.4 50.8))
+    (stroke (width 0) (type default))
+  )
+  (wire (pts (xy 25.4 40.64) (xy 30.48 40.64))
+    (stroke (width 0) (type default))
+  )
+  (wire (pts (xy 73.66 43.18) (xy 81.28 43.18))
+    (stroke (width 0) (type default))
+  )
+  (wire (pts (xy 73.66 17.78) (xy 81.28 17.78))
+    (stroke (width 0) (type default))
+  )
+  (wire (pts (xy 25.4 24.13) (xy 30.48 24.13))
     (stroke (width 0) (type default))
   )
@@
     (stroke (width 0) (type default))
   )
-  (wire (pts (xy 25.4 29.21) (xy 30.48 29.21))
-    (stroke (width 0) (type default))
-  )
-  (polyline (pts (xy 12.7 60.96) (xy 52.07 60.96))
-    (stroke (width 0) (type default))
-  )
-  (polyline (pts (xy 104.14 12.7) (xy 104.14 60.96))
-    (stroke (width 0) (type default))
-  )
-  (wire (pts (xy 25.4 43.18) (xy 30.48 43.18))
-    (stroke (width 0) (type default))
-  )
-  (wire (pts (xy 73.66 33.02) (xy 81.28 33.02))
-    (stroke (width 0) (type default))
-  )
-  (polyline (pts (xy 52.07 12.7) (xy 52.07 60.96))
-    (stroke (width 0) (type default))
-  )
-  (wire (pts (xy 73.66 38.1) (xy 81.28 38.1))
-    (stroke (width 0) (type default))
-  )
-  (wire (pts (xy 25.4 26.67) (xy 30.48 26.67))
-    (stroke (width 0) (type default))
-  )
-  (wire (pts (xy 25.4 48.26) (xy 25.4 50.8))
-    (stroke (width 0) (type default))
-  )
-  (wire (pts (xy 25.4 40.64) (xy 30.48 40.64))
-    (stroke (width 0) (type default))
-  )
-  (wire (pts (xy 73.66 43.18) (xy 81.28 43.18))
-    (stroke (width 0) (type default))
-  )
-  (wire (pts (xy 73.66 17.78) (xy 81.28 17.78))
-    (stroke (width 0) (type default))
-  )
-  (wire (pts (xy 25.4 24.13) (xy 30.48 24.13))
-    (stroke (width 0) (type default))
-  )
   (polyline (pts (xy 52.07 60.96) (xy 104.14 60.96))
     (stroke (width 0) (type default))
@@
     (effects (font (size 1.27 1.27)) (justify left bottom))
   )
+  (symbol (lib_id "power:GND") (at 74.93 54.61 0) (unit 1)
+    (in_bom yes) (on_board yes) (dnp no) (fields_autoplaced)
+    (property "Reference" "#PWR02" (at 74.93 60.96 0)
+      (effects (font (size 1.27 1.27)) hide)
+    )
+    (property "Value" "GND" (at 74.93 59.69 0)
+      (effects (font (size 1.27 1.27)))
+    )
+    (property "Footprint" "" (at 74.93 54.61 0)
+      (effects (font (size 1.27 1.27)) hide)
+    )
+    (property "Datasheet" "" (at 74.93 54.61 0)
+      (effects (font (size 1.27 1.27)) hide)
+    )
+    (pin "1")
+    (instances
+      (project "battery-balance-connector"
+        (path "/49388977-5cf7-4ef1-b585-6bfe2c096acf"
+          (reference "#PWR02") (unit 1)
+        )
+      )
+    )
+  )
   (symbol (lib_id "Connector_Generic:Conn_01x01") (at 86.36 38.1 0) (unit 1)
     (in_bom yes) (on_board yes) (dnp no) (fields_autoplaced)
@@
       (effects (font (size 1.27 1.27)) (justify left))
     )
-    (property "Footprint" "Connector_Wire:SolderWire-1sqmm_1x01_D1.4mm_OD2.7mm_Relief" (at 86.36 38.1 0)
+    (property "Footprint" "Connector_Wire:SolderWirePad_1x01_SMD_2x4mm_2.7mmRelief" (at 86.36 38.1 0)
       (effects (font (size 1.27 1.27)) hide)
     )
@@
       (effects (font (size 1.27 1.27)) (justify left))
     )
-    (property "Footprint" "Connector_Wire:SolderWire-1sqmm_1x01_D1.4mm_OD2.7mm_Relief" (at 86.36 48.26 0)
+    (property "Footprint" "Connector_Wire:SolderWirePad_1x01_SMD_2x4mm_2.7mmRelief" (at 86.36 48.26 0)
       (effects (font (size 1.27 1.27)) hide)
     )
@@
       (effects (font (size 1.27 1.27)) (justify left))
     )
-    (property "Footprint" "Connector_Wire:SolderWire-1sqmm_1x01_D1.4mm_OD2.7mm_Relief" (at 86.36 33.02 0)
+    (property "Footprint" "Connector_Wire:SolderWirePad_1x01_SMD_2x4mm_2.7mmRelief" (at 86.36 33.02 0)
       (effects (font (size 1.27 1.27)) hide)
     )
@@
     )
   )
-  (symbol (lib_id "power:GND") (at 74.93 54.61 0) (unit 1)
-    (in_bom yes) (on_board yes) (dnp no) (fields_autoplaced)
-    (property "Reference" "#PWR02" (at 74.93 60.96 0)
-      (effects (font (size 1.27 1.27)) hide)
-    )
-    (property "Value" "GND" (at 74.93 59.69 0)
-      (effects (font (size 1.27 1.27)))
-    )
-    (property "Footprint" "" (at 74.93 54.61 0)
-      (effects (font (size 1.27 1.27)) hide)
-    )
-    (property "Datasheet" "" (at 74.93 54.61 0)
-      (effects (font (size 1.27 1.27)) hide)
-    )
-    (pin "1")
-    (instances
-      (project "battery-balance-connector"
-        (path "/49388977-5cf7-4ef1-b585-6bfe2c096acf"
-          (reference "#PWR02") (unit 1)
-        )
-      )
-    )
-  )
   (symbol (lib_id "Connector_Generic:Conn_01x01") (at 86.36 22.86 0) (unit 1)
     (in_bom yes) (on_board yes) (dnp no) (fields_autoplaced)
@@
       (effects (font (size 1.27 1.27)) (justify left))
     )
-    (property "Footprint" "Connector_Wire:SolderWire-1sqmm_1x01_D1.4mm_OD2.7mm_Relief" (at 86.36 22.86 0)
+    (property "Footprint" "Connector_Wire:SolderWirePad_1x01_SMD_2x4mm_2.7mmRelief" (at 86.36 22.86 0)
       (effects (font (size 1.27 1.27)) hide)
     )
@@
       (effects (font (size 1.27 1.27)) (justify left))
     )
-    (property "Footprint" "Connector_Wire:SolderWire-1sqmm_1x01_D1.4mm_OD2.7mm_Relief" (at 86.36 27.94 0)
+    (property "Footprint" "Connector_Wire:SolderWirePad_1x01_SMD_2x4mm_2.7mmRelief" (at 86.36 27.94 0)
       (effects (font (size 1.27 1.27)) hide)
     )
@@
       (effects (font (size 1.27 1.27)) (justify left))
     )
-    (property "Footprint" "Connector_Wire:SolderWire-1sqmm_1x01_D1.4mm_OD2.7mm_Relief" (at 86.36 17.78 0)
+    (property "Footprint" "Connector_Wire:SolderWirePad_1x01_SMD_2x4mm_2.7mmRelief" (at 86.36 17.78 0)
       (effects (font (size 1.27 1.27)) hide)
     )
@@
       (effects (font (size 1.27 1.27)) (justify left))
     )
-    (property "Footprint" "Connector_Wire:SolderWire-1sqmm_1x01_D1.4mm_OD2.7mm_Relief" (at 86.36 43.18 0)
+    (property "Footprint" "Connector_Wire:SolderWirePad_1x01_SMD_2x4mm_2.7mmRelief" (at 86.36 43.18 0)
       (effects (font (size 1.27 1.27)) hide)
     )
@@
       (effects (font (size 1.27 1.27)) (justify left))
     )
-    (property "Footprint" "Connector_Wire:SolderWire-1sqmm_1x01_D1.4mm_OD2.7mm_Relief" (at 86.36 53.34 0)
-      (effects (font (size 1.27 1.27)) hide)
-    )
+    (property "Footprint" "Connector_Wire:SolderWirePad_1x01_SMD_2x4mm_2.7mmRelief" (at 86.36 53.34 0)
+      (effects (font (size 1.27 1.27)) hide)
+    )

Commit message: V1.0.1 - using vertical mounting and tweaked dimensions
Parts:
- J1, J2: footprint Connector_JST:JST_PH_S4B-PH-K_1x04_P2.00mm_Horizontal -> Connector_JST:JST_PH_B4B-PH-K_1x04_P2.00mm_Vertical
Changed lines of the file:
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@@
       (effects (font (size 1.27 1.27)) (justify left))
     )
-    (property "Footprint" "Connector_JST:JST_PH_S4B-PH-K_1x04_P2.00mm_Horizontal" (at 35.56 26.67 0)
+    (property "Footprint" "Connector_JST:JST_PH_B4B-PH-K_1x04_P2.00mm_Vertical" (at 35.56 26.67 0)
       (effects (font (size 1.27 1.27)) hide)
     )
@@
       (effects (font (size 1.27 1.27)) (justify left))
     )
-    (property "Footprint" "Connector_JST:JST_PH_S4B-PH-K_1x04_P2.00mm_Horizontal" (at 35.56 43.18 0)
+    (property "Footprint" "Connector_JST:JST_PH_B4B-PH-K_1x04_P2.00mm_Vertical" (at 35.56 43.18 0)
       (effects (font (size 1.27 1.27)) hide)
     )
